Commit message: feat: complete semantic target localization and approach pipeline

File: src/robot_description/urdf/gazebo.xacro (robot description, xacro)
@@ -18,5 +18,4 @@
         <mu2>0.01</mu2>
     </gazebo>
-<!--
     <gazebo reference="imu_link">
     <sensor name="imu_sensor" type="imu">
@@ -25,5 +24,5 @@
         <topic>imu</topic>
     </sensor>
-</gazebo> -->
+</gazebo>
 <gazebo reference="laser_link">
     <sensor name="gpu_lidar" type="gpu_lidar">
@@ -56,4 +55,23 @@
     </sensor>
 </gazebo>
+<gazebo reference="camera_link">
+    <sensor name="camera_sensor" type="camera">
+        <always_on>true</always_on>
+        <update_rate>30</update_rate>
+        <camera>
+            <horizontal_fov>1.047</horizontal_fov>
+            <image>
+                <width>640</width>
+                <height>480</height>
+                <format>R8G8B8</format>
+            </image>
+            <clip>
+                <near>0.1</near>
+                <far>20.0</far>
+            </clip>
+        </camera>
+        <topic>camera</topic>
+    </sensor>
+</gazebo>
     <!-- ============================= -->
     <!-- Gazebo Sim DiffDrive -->
@@ -69,5 +87,5 @@
             <topic>/cmd_vel</topic>
             <odom_topic>/odom</odom_topic>
-            <!-- tf_topic 已禁用：odom->base_footprint 由 odom_tf_broadcaster 发布，避免双发布冲突 -->
+            <!-- tf_topic 已禁用：odom->base_footprint 由 robot_localization EKF (publish_tf: true) 发布，避免双发布冲突 -->
             <!-- <tf_topic>/tf</tf_topic> -->
             <frame_id>odom</frame_id>

File: src/robot_description/urdf/robot_core.xacro (robot description, xacro)
@@ -44,5 +44,7 @@
         <inertial>
             <mass value="8.0"/>
-            <origin xyz="0 0 0"
+            <!-- COM 后移 5cm：避免激光/相机前移使总 COM 越过驱动轮轴
+                 支撑边界导致整车 nose-down 前倾（约 11.78°） -->
+            <origin xyz="-0.05 0 0"
                     rpy="0 0 0"/>
             <inertia
@@ -115,4 +117,39 @@
         <preserveFixedJoint>true</preserveFixedJoint>
     </gazebo>
+    <!-- Camera Link -->
+<link name="camera_link">
+    <visual>
+        <origin xyz="0 0 0" rpy="0 0 0"/>
+        <geometry>
+            <box size="0.08 0.08 0.06"/>
+        </geometry>
+        <material name="camera_gray">
+            <color rgba="0.2 0.2 0.2 1"/>
+        </material>
+    </visual>
+    <collision>
+        <origin xyz="0 0 0" rpy="0 0 0"/>
+        <geometry>
+            <box size="0.08 0.08 0.06"/>
+        </geometry>
+    </collision>
+    <inertial>
+        <mass value="0.05"/>
+        <origin xyz="0 0 0" rpy="0 0 0"/>
+        <inertia
+            ixx="0.00002"
+            iyy="0.00002"
+            izz="0.00002"
+            ixy="0.0"
+            ixz="0.0"
+            iyz="0.0"/>
+    </inertial>
+</link>
+<!-- Camera fixed joint -->
+<joint name="camera_joint" type="fixed">
+    <parent link="base_link"/>
+    <child link="camera_link"/>
+    <origin xyz="0.30 0 0.22" rpy="0 0 0"/>
+</joint>
     <!-- ============================= -->
     <!-- 轮子宏 -->
